File: 8bit-computer/inst-register.kicad_sch (KiCad schematic)
At the start: 20 parts, among them U13 74LS245, U14 74LS173, U15 74LS173

Commit message: cont. drawing CPU
Other:
- title: (none) -> IR (Instruction register)
