File: 8bit-computer/a-register.kicad_sch (KiCad schematic)
At the start: 20 parts, among them U7 74LS245, U8 74LS173, U9 74LS173

Commit message: designing register schematic
Parts:
- removed C11: 0.1µF, Capacitor_THT:C_Disc_D4.3mm_W1.9mm_P5.00mm, symbol Device:C
- removed D10, D11, D12, D13, D14, D15, D16, D17: RED, LED_THT:LED_D5.0mm, symbol Device:LED_ALT
- removed U9: 74LS173, Package_DIP:DIP-16_W7.62mm, symbol 74xx:74LS173
- added C1: 0.1µF, Capacitor_THT:C_Disc_D4.3mm_W1.9mm_P5.00mm, symbol Device:C
- added D10, D11, D12, D13, D14, D15, D16, D17: RED, LED_THT:LED_D5.0mm, symbol Device:LED
- added U10: 74LS173, Package_DIP:DIP-16_W7.62mm, symbol 74xx:74LS173
Connections:
- net A_0: now also U7.2 (A0), U8.3 (Q0), D17.2 (A)
- net A_1: now also U7.3 (A1), U8.4 (Q1), D16.2 (A)
- net A_2: now also U7.4 (A2), U8.5 (Q2), D15.2 (A)
- net A_3: now also U7.5 (A3), U8.6 (Q3), D14.2 (A)
- net A_4: now also U7.6 (A4), D13.2 (A), U10.3 (Q0)
- net A_5: now also U7.7 (A5), D12.2 (A), U10.4 (Q1)
- net A_6: now also U7.8 (A6), D11.2 (A), U10.5 (Q2)
- net A_7: now also U7.9 (A7), D10.2 (A), U10.6 (Q3)
- net BUS_0: now also U7.18 (B0), U10.11 (D3)
- net BUS_1: now also U7.17 (B1), U10.12 (D2)
- net BUS_2: now also U7.16 (B2), U10.13 (D1)
- net BUS_3: now also U7.15 (B3), U10.14 (D0)
- net BUS_4: now also U7.14 (B4), U8.11 (D3)
- net BUS_5: now also U7.13 (B5), U8.12 (D2)
- net BUS_6: now also U7.12 (B6), U8.13 (D1)
- net BUS_7: now also U7.11 (B7), U8.14 (D0)
- net CLK: now also U8.7 (Cp), U10.7 (Cp)
- net CLR: now also U8.15 (Mr), U10.15 (Mr)
- new net: D17.1 (K), R31.1
- new net: D10.1 (K), R24.1
- new net: D13.1 (K), R27.1
- new net: D12.1 (K), R26.1
- new net: D14.1 (K), R28.1
- new net: D11.1 (K), R25.1
- new net: D16.1 (K), R30.1
- new net: D15.1 (K), R29.1
- new net GND: C1.2, R24.2, R25.2, R26.2, R27.2, R28.2, R29.2, R30.2, R31.2, U10.1 (Oe1), U10.2 (Oe2), U10.8 (GND), U7.10 (GND), U8.1 (Oe1), U8.2 (Oe2), U8.8 (GND)
- new net VCC: C1.1, U10.16 (VCC), U7.1 (A->B), U7.20 (VCC), U8.16 (VCC)
- new net ~{AI}: U10.10 (E2), U10.9 (E1), U8.10 (E2), U8.9 (E1)
- new net ~{AO}: U7.19 (CE)
