File: 8bit-computer/alu.kicad_sch (KiCad schematic)
At the start: 30 parts, among them U16 74LS86, U17 74LS245, U18 74LS86, U19 74LS173, U20 74LS283, U21 74LS283, U22 74LS02, U23 74LS08

Commit message: starting alu
Parts:
- added unit 5 of U16
- added unit 5 of U18
Connections:
- net SU: now also U16.10, U16.13, U16.2, U16.5, U18.10, U18.13, U18.2, U18.5
- new net GND: U16.14 (VCC), U18.14 (VCC)
- new net VCC: U16.7 (GND), U18.7 (GND)

Commit message: impl. ALU
Parts:
- removed D34, D35: GREEN, LED_THT:LED_D5.0mm, symbol Device:LED_ALT
- removed D74, D75, D76, D77, D78, D79, D80, D81: RED, LED_THT:LED_D5.0mm, symbol Device:LED_ALT
- removed R48, R49, R92, R93, R94, R95, R96, R97, R98, R99: 220, Resistor_THT:R_Axial_DIN0207_L6.3mm_D2.5mm_P7.62mm_Horizontal, symbol Device:R
- removed U17: 74LS245, Package_DIP:DIP-20_W7.62mm, symbol 74xx:74LS245
- removed U20, U21: 74LS283, Package_DIP:DIP-16_W7.62mm, symbol 74xx:74LS283
- added D74, D75, D76, D77, D78, D79, D80, D81, D82, D83: LED, LED_THT:LED_D5.0mm, symbol Device:LED
- added R1, R10, R2, R3, R4, R5, R6, R7, R8, R9: 220, Resistor_THT:R_Axial_DIN0207_L6.3mm_D2.5mm_P7.62mm_Horizontal, symbol Device:R
- added U1, U2: 74LS283, Package_DIP:DIP-16_W7.62mm, symbol 74xx:74LS283
- added unit 5 of U22
- added unit 5 of U23
- added U3: 74LS245, Package_DIP:DIP-20_W7.62mm, symbol 74xx:74LS245
- C14, C15: footprint Capacitor_THT:C_Disc_D4.3mm_W1.9mm_P5.00mm -> (none)
Connections:
- net A_0: now also U2.12 (A4)
- net A_1: now also U2.14 (A3)
- net A_2: now also U2.3 (A2)
- net A_3: now also U2.5 (A1)
- net A_4: now also U1.12 (A4)
- net A_5: now also U1.14 (A3)
- net A_6: now also U1.3 (A2)
- net A_7: now also U1.5 (A1)
- net BUS_0: now also U3.18 (B0)
- net BUS_1: now also U3.17 (B1)
- net BUS_2: now also U3.16 (B2)
- net BUS_3: now also U3.15 (B3)
- net BUS_4: now also U3.14 (B4)
- net BUS_5: now also U3.13 (B5)
- net BUS_6: now also U3.12 (B6)
- net BUS_7: now also U3.11 (B7)
- net B_0: now also U18.12
- net B_1: now also U18.9
- net B_2: now also U18.4
- net B_3: now also U18.1
- net B_4: now also U16.12
- net B_5: now also U16.9
- net B_6: now also U16.4
- net B_7: now also U16.1
- net CF: now also U19.3 (Q0), R9.1
- net CLK: now also U19.7 (Cp)
- net CLR: now also U19.15 (Mr)
- net GND: now also C14.2, C15.2, U16.7 (GND), U18.7 (GND), U19.1 (Oe1), U19.2 (Oe2), D74.1 (K), D75.1 (K), D76.1 (K), D77.1 (K), D78.1 (K), D79.1 (K), D80.1 (K), D81.1 (K), D82.1 (K), D83.1 (K), U1.8 (GND), U2.8 (GND), U22.7 (GND), U23.7 (GND), U3.10 (GND); no longer U16.14 (VCC), U18.14 (VCC)
- net SU: now also U2.7 (C0)
- net VCC: now also C14.1, C15.1, U16.14 (VCC), U18.14 (VCC), U1.16 (VCC), U2.16 (VCC), U22.14 (VCC), U23.14 (VCC), U3.1 (A->B), U3.20 (VCC); no longer U16.7 (GND), U18.7 (GND)
- net ZF: now also U19.4 (Q1), R10.1
- net ~{EO}: now also U3.19 (CE)
- net B5: now reaches U16.8
- net B5: now also U1.15 (B3)
- net B1: now reaches U18.8
- net B1: now also U2.15 (B3)
- net B0: now reaches U18.11
- net B0: now also U2.11 (B4)
- net B7: now reaches U16.3
- net B7: now also U1.6 (B1)
- net B4: now reaches U16.11
- net B4: now also U1.11 (B4)
- net B3: now reaches U18.3
- net B3: now also U2.6 (B1)
- net B6: now reaches U16.6
- net B6: now also U1.2 (B2)
- net B2: now reaches U18.6
- net B2: now also U2.2 (B2)
- new net: D75.2 (A), R2.2
- new net: D82.2 (A), R9.2
- new net: D77.2 (A), R4.2
- new net: D81.2 (A), R8.2
- new net: D74.2 (A), R1.2
- new net: U23.10, U23.6
- new net: U19.13 (D1), U23.8
- new net: U23.3, U23.9
- new net: U1.7 (C0), U2.9 (C4)
- new net: U1.9 (C4), U19.14 (D0)
- new net: D79.2 (A), R6.2
- new net: D78.2 (A), R5.2
- new net: U22.1, U23.1
- new net: U22.10, U23.4
- new net: U22.13, U23.5
- new net: D80.2 (A), R7.2
- new net: U22.4, U23.2
- new net: D76.2 (A), R3.2
- new net: D83.2 (A), R10.2
- new net R0: R1.1, U2.10 (S4), U22.12, U3.2 (A0)
- new net R1: R2.1, U2.13 (S3), U22.11, U3.3 (A1)
- new net R2: R3.1, U2.1 (S2), U22.9, U3.4 (A2)
- new net R3: R4.1, U2.4 (S1), U22.8, U3.5 (A3)
- new net R4: R5.1, U1.10 (S4), U22.6, U3.6 (A4)
- new net R5: R6.1, U1.13 (S3), U22.5, U3.7 (A5)
- new net R6: R7.1, U1.1 (S2), U22.3, U3.8 (A6)
- new net R7: R8.1, U1.4 (S1), U22.2, U3.9 (A7)
- new net ~{FI}: U19.10 (E2), U19.9 (E1)
Other:
- moved on the sheet: U16A, U16B, U16C, U16D, U18A, U18B, U18C, U18D

Commit message: cont. 8bit schematics
Parts:
- removed unit 5 of U16
- removed unit 5 of U18
- removed unit 5 of U22
- removed unit 5 of U23
- removed unit 4 of U23
Connections:
- no-connect marks 7 -> 4
Other:
- title: (none) -> Arithmetic Logic Unit (ALU)
- moved on the sheet: C14, C15
