File: 8bit-computer/control.kicad_sch (KiCad schematic)
At the start: 59 parts, among them SW8 Reset, U47 28C16, U48 74LS161, U49 74LS04, U50 74LS138, U51 74LS00, U52 28C16, U53 74LS04

Commit message: cont. drawing CPU
Connections:
- net VCC: now also R67.1, R68.1, R69.1, R70.1, R71.1
- net GND: now reaches U47.1 (A7), U47.18 (~CE), U47.19 (A10), U47.20 (~OE), U52.18 (~CE), U52.19 (A10), U52.20 (~OE)
- net GND: now also R72.2, R73.2, R74.2, R75.2, R76.2, R77.2, R78.2, R79.2, R80.2, R81.2, R82.2, R83.2, R84.2, R85.2, R86.2, R87.2, R88.2, R89.2, R90.2, R91.2
Changed lines of the file:
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@@
 	(generator "eeschema")
 	(generator_version "10.0")
-	(paper "USLetter")
+	(paper "A3")
 	(junction
 		(at 93.98 193.04)

Commit message: cont. 8bit schematics
Parts:
- removed C22, C23: 0.1µF, Capacitor_THT:C_Disc_D4.3mm_W1.9mm_P5.00mm, symbol Device:C
- removed D50, D52, D53, D55, D56: GREEN, LED_THT:LED_D5.0mm, symbol Device:LED_ALT
- removed D51, D54, D57: RED, LED_THT:LED_D5.0mm, symbol Device:LED_ALT
- removed D58, D59, D60, D61, D62, D63, D64, D65, D66, D67, D68, D69, D70, D71, D72, D73: BLUE, LED_THT:LED_D5.0mm, symbol Device:LED_ALT
- removed R67, R68, R69, R70, R71, R72, R73, R74, R76, R77, R78, R79, R80, R81, R82, R83, R84, R85, R86, R87, R88, R89, R90, R91: 220, Resistor_THT:R_Axial_DIN0207_L6.3mm_D2.5mm_P7.62mm_Horizontal, symbol Device:R
- removed SW8: Reset, Button_Switch_THT:SW_PUSH_6mm_H5mm, symbol Switch:SW_Push
- removed U48: 74LS161, Package_DIP:DIP-16_W7.62mm, symbol 74xx:74LS161
- removed U49, U53: 74LS04, Package_DIP:DIP-14_W7.62mm, symbol 74xx:74LS04
- removed U50: 74LS138, Package_DIP:DIP-16_W7.62mm, symbol 74xx:74LS138
- added C7, C8: 0.1µF, Capacitor_THT:C_Disc_D4.3mm_W1.9mm_P5.00mm, symbol Device:C
- added D18, D19, D20, D21, D22, D23, D24, D25: LED, LED_THT:LED_D5.0mm, symbol Device:LED
- added R32, R33, R34, R35, R36, R37, R38, R39: 220, Resistor_THT:R_Axial_DIN0207_L6.3mm_D2.5mm_P7.62mm_Horizontal, symbol Device:R
- added SW3: SW_Push, Button_Switch_THT:SW_PUSH_6mm_H5mm, symbol Switch:SW_Push
- added U11, U9: 74LS04, Package_DIP:DIP-14_W7.62mm, symbol 74xx:74LS04
- added U12: 74LS138, Package_DIP:DIP-16_W7.62mm, symbol 74xx:74LS138
- added U13: 74LS161, Package_DIP:DIP-16_W7.62mm, symbol 74xx:74LS161
Connections:
- net CLR: now also U51.8
- net GND: now also U47.12 (GND), U52.12 (GND), C7.2, C8.2, D18.1 (K), D19.1 (K), D20.1 (K), D21.1 (K), D22.1 (K), D23.1 (K), D24.1 (K), D25.1 (K), U12.4 (E1), U12.5 (E2)
- net VCC: now also U47.24 (VCC), U52.24 (VCC), C7.1, C8.1, SW3.2, U12.6 (E3), U13.10 (CET), U13.7 (CEP), U13.9 (~{PE})
- net at R75.1: now also U51.12, U51.13, SW3.1
- net at U52.10 (D1): now also U11.9
- net at U52.11 (D2): now also U11.5
- net at U52.15 (D5): now also U11.3
- net at U52.17 (D7): now also U11.1
- net at U47.6 (A2), U52.6 (A2): now also R37.2, U12.3 (A2), U13.12 (Q2)
- net at U47.7 (A1), U52.7 (A1): now also R38.2, U12.2 (A1), U13.13 (Q1)
- net at U47.8 (A0), U52.8 (A0): now also R39.2, U12.1 (A0), U13.14 (Q0)
- net at U52.9 (D0): now also U11.11
- net at U47.10 (D1): now also U9.11
- net at U47.11 (D2): now also U9.9
- net at U47.13 (D3): now also U9.5
- net at U47.14 (D4): now also U9.3
- net at U47.16 (D6): now also U9.1
- net at U47.9 (D0): now also U9.13
- new net: D21.2 (A), R35.1
- new net: R35.2, U12.12 (O3)
- new net: D24.2 (A), R38.1
- new net: D22.2 (A), R36.1
- new net: R36.2, U12.11 (O4)
- new net: D23.2 (A), R37.1
- new net: D18.2 (A), R32.1
- new net: D25.2 (A), R39.1
- new net: U51.1, U51.2, U51.6
- new net: U13.1 (~{MR}), U51.3
- new net: D20.2 (A), R34.1
- new net: R32.2, U12.15 (O0)
- new net: U12.10 (O5), U51.5
- new net: D19.2 (A), R33.1
- new net: R33.2, U12.14 (O1)
- new net: R34.2, U12.13 (O2)
- new net ~{AI}: U9.10
- new net ~{AO}: U9.12
- new net ~{BI}: U11.4
- new net ~{CLK}: U13.2 (CP)
- new net ~{CLR}: U51.10, U51.11, U51.4, U51.9
- new net ~{CO}: U11.6
- new net ~{EO}: U11.2
- new net ~{FI}: U11.10
- new net ~{II}: U9.8
- new net ~{IO}: U9.6
- new net ~{J}: U11.8
- new net ~{MI}: U9.2
- new net ~{RO}: U9.4
- no-connect marks 10 -> 8
Other:
- title: (none) -> Control Unit (CU)
