File: 8bit-computer/program-counter.kicad_sch (KiCad schematic)
At the start: 11 parts, among them U35 74LS161, U36 74LS245

Commit message: cont. drawing CPU
Parts:
- removed D82, D83, D84, D85: GREEN, LED_THT:LED_D5.0mm, symbol Device:LED_ALT
- added D82, D83, D84, D85: GREEN, LED_THT:LED_D5.0mm, symbol Device:LED_Filled
- C19: value 0.1µF -> 100nF
Connections:
- net BUS_0: now also U35.3 (D0), U36.9 (A7)
- net BUS_1: now also U35.4 (D1), U36.8 (A6)
- net BUS_2: now also U35.5 (D2), U36.7 (A5)
- net BUS_3: now also U35.6 (D3), U36.6 (A4)
- net CE: now also U35.10 (CET), U35.7 (CEP)
- net CLK: now also U35.2 (CP)
- new net: D82.1 (K), R100.2
- new net: D82.2 (A), U35.11 (Q3), U36.14 (B4)
- new net: D83.1 (K), R101.2
- new net: D83.2 (A), U35.12 (Q2), U36.13 (B5)
- new net: D84.1 (K), R102.2
- new net: D85.1 (K), R103.2
- new net: D84.2 (A), U35.13 (Q1), U36.12 (B6)
- new net: D85.2 (A), U35.14 (Q0), U36.11 (B7)
- new net GND: C19.2, R100.1, R101.1, R102.1, R103.1, U35.8 (GND), U36.1 (A->B), U36.10 (GND)
- new net VCC: C19.1, U35.16 (VCC), U36.20 (VCC)
- new net ~{CLR}: U35.1 (~{MR})
- new net ~{CO}: U36.19 (CE)
- new net ~{J}: U35.9 (~{PE})
Other:
- title: (none) -> PC (Program Counter)

Commit message: cont. 8bit schematics
Other:
- title: PC (Program Counter) -> Program Counter (PC)
Changed lines of the file:
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@@
 	(paper "A4")
 	(title_block
-		(title "PC (Program Counter)")
+		(title "Program Counter (PC)")
 		(date "2026-05-12")
 		(comment 1 "is currently executing.")
