File: 8bit-computer/mar.kicad_sch (KiCad schematic)
At the start: 17 parts, among them SW5 SW_DIP_x04, SW6 SW_SPDT, U33 74LS157, U34 74LS173

Commit message: cont. 8bit schematics
Other:
- title: (none) -> Memory Address Register (MAR)
Changed lines of the file:
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@@
 	(generator_version "10.0")
 	(paper "A4")
+	(title_block
+		(title "Memory Address Register (MAR)")
+		(date "2026-05-15")
+	)
 	(junction
 		(at 88.9 93.98)

Commit message: memory address register
Parts:
- removed D44, D45, D46, D47: YELLOW, LED_THT:LED_D5.0mm, symbol Device:LED_ALT
- removed D48: RED, LED_THT:LED_D5.0mm, symbol Device:LED_ALT
- removed D49: GREEN, LED_THT:LED_D5.0mm, symbol Device:LED_ALT
- removed R59, R60, R61, R62: 220, Resistor_THT:R_Axial_DIN0207_L6.3mm_D2.5mm_P7.62mm_Horizontal, symbol Device:R
- removed R63, R64: 1K, Resistor_THT:R_Axial_DIN0207_L6.3mm_D2.5mm_P7.62mm_Horizontal, symbol Device:R
- removed SW5: SW_DIP_x04, Button_Switch_THT:SW_DIP_SPSTx04_Slide_9.78x12.34mm_W7.62mm_P2.54mm, symbol Switch:SW_DIP_x04
- removed SW6: SW_SPDT, 8bit-custom-footprints:DPDT-pushbutton, symbol Switch:SW_SPDT
- removed U33: 74LS157, Package_DIP:DIP-16_W7.62mm, symbol 74xx:74LS157
- removed U34: 74LS173, Package_DIP:DIP-16_W7.62mm, symbol 74xx:74LS173
- added SW4: SW_DIP_x04, Button_Switch_THT:SW_DIP_SPSTx04_Slide_9.78x12.34mm_W7.62mm_P2.54mm, symbol Switch:SW_DIP_x04
- added SW5: SW_SPDT, symbol Switch:SW_SPDT
- added U14: 74LS173, Package_DIP:DIP-16_W7.62mm, symbol 74xx:74LS173
- added U15: 74LS157, symbol 74xx:74LS157
Connections:
- net A0: now also U15.12 (Zd)
- net A1: now also U15.9 (Zc)
- net A2: now also U15.7 (Zb)
- net A3: now also U15.4 (Za)
- net BUS_0: now also U14.14 (D0)
- net BUS_1: now also U14.13 (D1)
- net BUS_2: now also U14.12 (D2)
- net BUS_3: now also U14.11 (D3)
- net CLK: now also U14.7 (Cp)
- net CLR: now also U14.15 (Mr)
- net PROG: now also SW5.1 (A), U15.1 (S)
- new net: U14.5 (Q2), U15.10 (I1c)
- new net: SW4.3, U15.11 (I0c)
- new net: U14.6 (Q3), U15.13 (I1d)
- new net: SW4.4, U15.14 (I0d)
- new net: SW4.1, U15.2 (I0a)
- new net: U14.3 (Q0), U15.3 (I1a)
- new net: SW4.2, U15.5 (I0b)
- new net: U14.4 (Q1), U15.6 (I1b)
- new net GND: C18.2, SW4.5, SW4.6, SW4.7, SW4.8, SW5.2 (B), U14.1 (Oe1), U14.2 (Oe2), U14.8 (GND), U15.15 (E), U15.8 (GND)
- new net VCC: C18.1, U14.16 (VCC), U15.16 (VCC)
- new net ~{MI}: U14.10 (E2), U14.9 (E1)
- no-connect marks 0 -> 1
