File: 8bit-computer/ram.kicad_sch (KiCad schematic)
At the start: 31 parts, among them SW3 SW_DIP_x08, SW4 SW_Push, U24 74189, U25 74189, U26 74LS157, U27 74LS157, U28 74LS04, U29 74LS04, U30 74LS245, U31 74LS00, U32 74LS157

Commit message: cont. drawing CPU
Other:
- title: (none) -> Random Access Memory (RAM)
- moved on the sheet: U24, U25

Commit message: drawing ram
Parts:
- removed C16, C17: 0.1µF, Capacitor_THT:C_Disc_D4.3mm_W1.9mm_P5.00mm, symbol Device:C
- removed C7: 0.01µF, Capacitor_THT:C_Disc_D4.3mm_W1.9mm_P5.00mm, symbol Device:C
- removed D36, D37, D38, D39, D40, D41, D42, D43: RED, LED_THT:LED_D5.0mm, symbol Device:LED_ALT
- removed R50, R51, R52, R53, R54, R55, R56, R57: 220, Resistor_THT:R_Axial_DIN0207_L6.3mm_D2.5mm_P7.62mm_Horizontal, symbol Device:R
- removed R58: 1K, Resistor_THT:R_Axial_DIN0207_L6.3mm_D2.5mm_P7.62mm_Horizontal, symbol Device:R
- removed SW3: SW_DIP_x08, Button_Switch_THT:SW_DIP_SPSTx08_Slide_9.78x22.5mm_W7.62mm_P2.54mm, symbol Switch:SW_DIP_x08
- removed SW4: SW_Push, Button_Switch_THT:SW_PUSH_6mm_H5mm, symbol Switch:SW_Push
- removed U24: 74189, Package_DIP:DIP-16_W7.62mm, symbol 8bit-computer:74189
- removed U26, U27, U32: 74LS157, Package_DIP:DIP-16_W7.62mm, symbol 74xx:74LS157
- removed U28, U29: 74LS04, Package_DIP:DIP-14_W7.62mm, symbol 74xx:74LS04
- removed U30: 74LS245, Package_DIP:DIP-20_W7.62mm, symbol 74xx:74LS245
- removed U31: 74LS00, Package_DIP:DIP-14_W7.62mm, symbol 74xx:74LS00
- added C10, C11, C9: 0.1µF, symbol Device:C
- added R40: 1K, symbol Device:R
- added SW6: SW_DIP_x08, Button_Switch_THT:SW_DIP_SPSTx08_Slide_9.78x22.5mm_W7.62mm_P2.54mm, symbol Switch:SW_DIP_x08
- added SW7: SW_Push, symbol Switch:SW_Push
- added U17, U20: 74LS04, Package_DIP:DIP-14_W7.62mm, symbol 74xx:74LS04
- added U21: 74LS245, Package_DIP:DIP-20_W7.62mm, symbol 74xx:74LS245
- added U24: 74LS157, Package_DIP:DIP-16_W7.62mm, symbol 74xx:74LS157
- added U26: 74F189, Package_DIP:DIP-16_W7.62mm, symbol 8bit-computer:74189
- added U27: 74LS00, symbol 74xx:74LS00
- added U28, U29: 74LS157, symbol 74xx:74LS157
- U25: value 74189 -> 74F189
Connections:
- net A0: now also U26.1 (A0)
- net A1: now also U26.15 (A1)
- net A2: now also U26.14 (A2)
- net A3: now also U26.13 (A3)
- net BUS_0: now also U21.11 (B7), U21.18 (B0), U28.2 (I0a), U29.14 (I0d)
- net BUS_1: now also U21.12 (B6), U21.17 (B1), U28.5 (I0b), U29.11 (I0c)
- net BUS_2: now also U21.13 (B5), U21.16 (B2), U28.11 (I0c), U29.5 (I0b)
- net BUS_3: now also U21.14 (B4), U21.15 (B3), U28.14 (I0d), U29.2 (I0a)
- net CLK: now also C11.1
- net PROG: now also U28.1 (S), U29.1 (S)
- net RI: now also U27.1
- net at U25.3 (~{WE}): now also U24.9 (Zc), U26.3 (~{WE})
- net DI5: now reaches U25.10 (D3)
- net DI5: now also U29.7 (Zb)
- net ~{D}4: now reaches U25.11 (O4)
- net ~{D}4: now also U17.11
- net DI4: now reaches U25.12 (D4)
- net DI4: now also U29.4 (Za)
- net VCC: now reaches U25.16 (VCC)
- net VCC: now also C10.1, C9.1, U21.1 (A->B), U21.20 (VCC), U24.16 (VCC), U26.16 (VCC), U28.16 (VCC), U29.16 (VCC)
- net GND: now reaches U25.2 (~{CS})
- net GND: now also U25.8 (GND), C10.2, C9.2, R40.2, SW6.1, SW6.2, SW6.3, SW6.4, SW6.5, SW6.6, SW6.7, SW6.8, SW7.1, U21.10 (GND), U24.8 (GND), U26.2 (~{CS}), U26.8 (GND), U28.8 (GND), U29.8 (GND)
- net DI7: now reaches U25.4 (D1)
- net DI7: now also U29.12 (Zd)
- net ~{D}7: now reaches U25.5 (O1)
- net ~{D}7: now also U17.1
- net DI6: now reaches U25.6 (D2)
- net DI6: now also U29.9 (Zc)
- net ~{D}6: now reaches U25.7 (O2)
- net ~{D}6: now also U17.3
- net ~{D}5: now reaches U25.9 (O3)
- net ~{D}5: now also U17.13
- new net: U24.10 (I1c), U27.3
- new net: SW7.2, U24.11 (I0c)
- new net: SW6.14, U28.10 (I1c)
- new net: SW6.13, U28.13 (I1d)
- new net: SW6.16, U28.3 (I1a)
- new net: SW6.15, U28.6 (I1b)
- new net: SW6.10, U29.10 (I1c)
- new net: SW6.11, U29.6 (I1b)
- new net: SW6.12, U29.3 (I1a)
- new net: SW6.9, U29.13 (I1d)
- new net: C11.2, R40.1, U27.2
- new net D0: U20.2, U21.2 (A0)
- new net D1: U20.4, U21.3 (A1)
- new net D2: U17.6, U21.4 (A2)
- new net D3: U17.8, U21.5 (A3)
- new net D4: U17.10, U21.6 (A4)
- new net D5: U17.12, U21.7 (A5)
- new net D6: U17.4, U21.8 (A6)
- new net D7: U17.2, U21.9 (A7)
- new net DI0: U26.12 (D4), U28.4 (Za)
- new net DI1: U26.10 (D3), U28.7 (Zb)
- new net DI2: U26.6 (D2), U28.9 (Zc)
- new net DI3: U26.4 (D1), U28.12 (Zd)
- new net ~{D}0: U20.1, U26.11 (O4)
- new net ~{D}1: U20.3, U26.9 (O3)
- new net ~{D}2: U17.5, U26.7 (O2)
- new net ~{D}3: U17.9, U26.5 (O1)
- new net ~{RO}: U21.19 (CE)
- new net ~{Ro}: U28.15 (E), U29.15 (E)
- no-connect marks 26 -> 11
