File: 8bit-computer/output.kicad_sch (KiCad schematic)
At the start: 18 parts, among them SW7 SW_SPDT, U37 74LS76, U38 74LS139, U39 LM555, U40 7SEGMENT_CC, U41 7SEGMENT_CC, U42 7SEGMENT_CC, U43 7SEGMENT_CC, U44 74LS273, U45 28C16, U46 74LS08

Commit message: drawing 7-Segment output
Parts:
- removed C20, C21: 0.1µF, Capacitor_THT:C_Disc_D4.3mm_W1.9mm_P5.00mm, symbol Device:C
- removed C8, C9: 0.01µF, Capacitor_THT:C_Disc_D4.3mm_W1.9mm_P5.00mm, symbol Device:C
- removed R104: 10k, Resistor_THT:R_Axial_DIN0207_L6.3mm_D2.5mm_P7.62mm_Horizontal, symbol Device:R
- removed R65: 1K, Resistor_THT:R_Axial_DIN0207_L6.3mm_D2.5mm_P7.62mm_Horizontal, symbol Device:R
- removed R66: 100K, Resistor_THT:R_Axial_DIN0207_L6.3mm_D2.5mm_P7.62mm_Horizontal, symbol Device:R
- removed SW7: SW_SPDT, 8bit-custom-footprints:DPDT-pushbutton, symbol Switch:SW_SPDT
- removed U38: 74LS139, Package_DIP:DIP-16_W7.62mm, symbol 74xx:74LS139
- removed U39: LM555, Package_DIP:DIP-8_W7.62mm, symbol Timer:LM555xN
- removed U40, U41, U42, U43: 7SEGMENT_CC, Display_7Segment:7SegmentLED_LTS6760_LTS6780, symbol 8bit-computer:7SEGMENT_CC
- removed U44: 74LS273, Package_DIP:DIP-20_W7.62mm, symbol 74xx:74LS273
- removed U45: 28C16, Package_DIP:DIP-24_W15.24mm_Socket, symbol 8bit-computer:28C16
- removed U46: 74LS08, Package_DIP:DIP-14_W7.62mm, symbol 74xx:74LS08
- added C12, C13: 0.1µF, symbol Device:C
- added C16, C17: 0.01µF, symbol Device:C
- added R41: 10k, symbol Device:R
- added R42: 1k, symbol Device:R
- added R43: 100k, symbol Device:R
- added SW8: SW_SPDT, symbol Switch:SW_SPDT
- added U30: 28C16, symbol 8bit-computer:28C16
- added U31: 74LS139, symbol 74xx:74LS139
- added U32: 74LS273, symbol 74xx:74LS273
- added U33: 74LS08, symbol 74xx:74LS08
- added U34: CA56-12EWA, Display_7Segment:CA56-12EWA, symbol Display_Character:CA56-12EWA
- added U38: LM555xN, Package_DIP:DIP-8_W7.62mm, symbol Timer:LM555xN
- U37: footprint Package_DIP:DIP-16_W7.62mm -> (none)
Connections:
- net BUS_0: now also U32.3 (D0)
- net BUS_1: now also U32.4 (D1)
- net BUS_2: now also U32.7 (D2)
- net BUS_3: now also U32.8 (D3)
- net BUS_4: now also U32.13 (D4)
- net BUS_5: now also U32.14 (D5)
- net BUS_6: now also U32.17 (D6)
- net BUS_7: now also U32.18 (D7)
- net CLK: now also U33.2
- net OI: now also U33.1
- new net: R42.2, R43.1, U38.7 (DISCH)
- new net: U37.1 (C), U38.3 (OUT)
- new net: U31.2 (A0), U37.14 (~{Q}), U37.6 (C)
- new net: U30.1 (A7), U32.19 (Q7)
- new net: U30.10 (D1), U34.7 (b)
- new net: U30.11 (D2), U34.4 (c)
- new net: U30.13 (D3), U34.2 (d)
- new net: U30.14 (D4), U34.1 (e)
- new net: U30.15 (D5), U34.10 (f)
- new net: U30.16 (D6), U34.5 (g)
- new net: U30.17 (D7), U34.3 (DPX)
- new net: SW8.2 (B), U30.19 (A10)
- new net: U30.2 (A6), U32.16 (Q6)
- new net: U30.3 (A5), U32.15 (Q5)
- new net: U30.4 (A4), U32.12 (Q4)
- new net: U30.5 (A3), U32.9 (Q3)
- new net: U30.6 (A2), U32.6 (Q2)
- new net: U30.7 (A1), U32.5 (Q1)
- new net: U30.8 (A0), U32.2 (Q0)
- new net: U30.9 (D0), U34.11 (a)
- new net: U31.3 (A1), U37.10 (~{Q})
- new net: C16.1, R43.2, U38.2 (TRIG), U38.6 (THRES)
- new net: C17.1, U38.5 (CONT)
- new net: U32.11 (Cp), U33.3
- new net: R41.1, SW8.3 (C)
- new net CA0: U31.4 (O0), U34.6 (CA4)
- new net CA1: U31.5 (O1), U34.8 (CA3)
- new net CA2: U31.6 (O2), U34.9 (CA2)
- new net CA3: U31.7 (O3), U34.12 (CA1)
- new net GND: C12.2, C13.2, C16.2, C17.2, R41.2, U30.12 (GND), U30.18 (~{CE}), U30.20 (~{OE}), U31.1 (E), U38.1 (GND)
- new net VCC: C12.1, C13.1, R42.1, SW8.1 (A), U30.21 (~{WE}), U30.24 (VCC), U37.12 (K), U37.16 (K), U37.2 (~{S}), U37.3 (~{R}), U37.4 (J), U37.7 (~{S}), U37.8 (~{R}), U37.9 (J), U38.8 (VCC)
- new net ~{CLR}: U32.1 (~{Mr})
- no-connect marks 19 -> 3
Other:
- title: (none) -> Output
